Commit message: Fixed mtm urdf file to correctly display parallel linkage

File: dvrk_model/model/mtm.urdf.xacro (robot description, xacro)
@@ -112,20 +112,20 @@
       </inertial>
     </link>
-    <!-- <link name="${prefix}front_parallel_link"> -->
-    <!--   <visual> -->
-    <!--     <geometry> -->
-    <!--       <mesh filename="package://dvrk_model/meshes/mtm/Link.dae"/> -->
-    <!--     </geometry> -->
-    <!--   </visual> -->
-    <!--   <collision> -->
-    <!--     <geometry> -->
-    <!--       <mesh filename="package://dvrk_model/meshes/mtm/Link.STL"/> -->
-    <!--     </geometry> -->
-    <!--   </collision> -->
-    <!--   <inertial> -->
-    <!--     <mass value="0.8"/> -->
-    <!--     <inertia ixx="8.0" ixy="0.0" ixz="0.0" iyy="8.0" iyz="0.0" izz="8.0"/> -->
-    <!--   </inertial>  -->
-    <!-- </link> -->
+     <link name="${prefix}front_parallel_link"> -->
+       <visual>
+         <geometry>
+           <mesh filename="package://dvrk_model/meshes/mtm/Link.dae"/> -->
+         </geometry>
+       </visual>
+       <collision>
+         <geometry>
+           <mesh filename="package://dvrk_model/meshes/mtm/Link.STL"/> -->
+         </geometry>
+       </collision>
+       <inertial>
+         <mass value="0.8"/>
+         <inertia ixx="8.0" ixy="0.0" ixz="0.0" iyy="8.0" iyz="0.0" izz="8.0"/> -->
+       </inertial>
+     </link>
     <joint name="${prefix}shoulder_pitch_joint" type="revolute">
       <parent link="${prefix}outer_yaw_link"/>
@@ -139,7 +139,7 @@
     </joint>
     <joint name="${prefix}shoulder_pitch_parallel_joint" type="revolute">
-      <parent link="${prefix}outer_yaw_link"/>
+      <parent link="${prefix}back_parallel_link"/>
       <child link="${prefix}top_parallel_link"/>
-      <origin rpy="${-PI/2} ${PI} 0" xyz="0 .065 -.19037"/>
+      <origin rpy="0 0 ${-PI/2}" xyz="0 0 0.065"/>
       <axis xyz="0 0 1"/>
       <!--rotates about  x axis-->
@@ -147,14 +147,15 @@
       <limit effort="100.0" lower="${-PI/2}" upper="${PI/2}" velocity="10"/>
       <joint_properties damping="1.0" friction="0.0"/>
-      <mimic joint="${prefix}shoulder_pitch_joint" multiplier="1"/>
-    </joint>
-    <!-- <joint name="${prefix}elbow_pitch_parallel_joint" type="revolute"> -->
-    <!--   <parent link="${prefix}top_parallel_link"/> -->
-    <!--   <child link="${prefix}front_parallel_link"/> -->
-    <!--   <origin rpy="0 0 0" xyz=".1011 0 -0.03"/> -->
-    <!--   <axis xyz="0 0 1"/> -->
-    <!--   <limit effort="100.0" lower="${-PI/4}" upper="${PI/4}" velocity="10"/> -->
-    <!--   <joint_properties damping="1.0" friction="0.0"/> -->
-    <!-- </joint> -->
+      <mimic joint="${prefix}elbow_pitch_joint" multiplier="1"/>
+    </joint>
+    <joint name="${prefix}elbow_pitch_parallel_joint" type="revolute">
+       <parent link="${prefix}top_parallel_link"/>
+       <child link="${prefix}front_parallel_link"/>
+       <origin rpy="0 0 0" xyz=".1011 0 -0.03"/>
+       <axis xyz="0 0 1"/>
+       <limit effort="100.0" lower="${-PI/4}" upper="${PI/4}" velocity="10"/>
+       <joint_properties damping="1.0" friction="0.0"/>
+       <mimic joint="${prefix}elbow_pitch_joint" multiplier="-1"/>
+     </joint>
     <joint name="${prefix}elbow_pitch_joint" type="revolute">
       <parent link="${prefix}back_parallel_link"/>

Commit message: Added gazebo control plugin to mtm.urdf.xacro file

File: dvrk_model/model/mtm.urdf.xacro (robot description, xacro)
@@ -298,7 +298,17 @@
       </inertial>
     </link>
+  <transmission name="tran1">
+    <type>transmission_interface/SimpleTransmission</type>
+    <joint name="${prefix}outer_yaw_joint"/>
+    <actuator name="motor1">
+      <hardwareInterface>EffortJointInterface</hardwareInterface>
+      <mechanicalReduction>1</mechanicalReduction>
+    </actuator>
+  </transmission>
+  <gazebo>
+    <plugin name="gazebo_ros_control" filename="libgazebo_ros_control.so">
+      <robotNamespace>/mtm</robotNamespace>
+    </plugin>
+  </gazebo>
   </xacro:macro>
-  <gazebo>
-    <plugin name="dv_adnan_controller" filename="libdv_adnan_controller.so" />
-  </gazebo>
 </robot>

Commit message: Added custom gazebo controllers for all the joints

File: dvrk_model/model/mtm.urdf.xacro (robot description, xacro)
@@ -112,20 +112,20 @@
       </inertial>
     </link>
-     <link name="${prefix}front_parallel_link"> -->
+     <!--link name="${prefix}front_parallel_link">
        <visual>
          <geometry>
-           <mesh filename="package://dvrk_model/meshes/mtm/Link.dae"/> -->
+           <mesh filename="package://dvrk_model/meshes/mtm/Link.dae"/>
          </geometry>
        </visual>
        <collision>
          <geometry>
-           <mesh filename="package://dvrk_model/meshes/mtm/Link.STL"/> -->
+           <mesh filename="package://dvrk_model/meshes/mtm/Link.STL"/>
          </geometry>
        </collision>
        <inertial>
          <mass value="0.8"/>
-         <inertia ixx="8.0" ixy="0.0" ixz="0.0" iyy="8.0" iyz="0.0" izz="8.0"/> -->
+         <inertia ixx="8.0" ixy="0.0" ixz="0.0" iyy="8.0" iyz="0.0" izz="8.0"/>
        </inertial>
-     </link>
+     </link-->
     <joint name="${prefix}shoulder_pitch_joint" type="revolute">
       <parent link="${prefix}outer_yaw_link"/>
@@ -149,5 +149,5 @@
       <mimic joint="${prefix}elbow_pitch_joint" multiplier="1"/>
     </joint>
-    <joint name="${prefix}elbow_pitch_parallel_joint" type="revolute">
+    <!--joint name="${prefix}elbow_pitch_parallel_joint" type="revolute">
        <parent link="${prefix}top_parallel_link"/>
        <child link="${prefix}front_parallel_link"/>
@@ -157,5 +157,5 @@
        <joint_properties damping="1.0" friction="0.0"/>
        <mimic joint="${prefix}elbow_pitch_joint" multiplier="-1"/>
-     </joint>
+     </joint-->
     <joint name="${prefix}elbow_pitch_joint" type="revolute">
       <parent link="${prefix}back_parallel_link"/>
@@ -302,4 +302,52 @@
     <joint name="${prefix}outer_yaw_joint"/>
     <actuator name="motor1">
+      <hardwareInterface>EffortJointInterface</hardwareInterface>
+      <mechanicalReduction>1</mechanicalReduction>
+    </actuator>
+  </transmission>
+  <transmission name="tran2">
+    <type>transmission_interface/SimpleTransmission</type>
+    <joint name="${prefix}shoulder_pitch_joint"/>
+    <actuator name="motor2">
+      <hardwareInterface>EffortJointInterface</hardwareInterface>
+      <mechanicalReduction>1</mechanicalReduction>
+    </actuator>
+  </transmission>
+  <transmission name="tran3">
+    <type>transmission_interface/SimpleTransmission</type>
+    <joint name="${prefix}elbow_pitch_joint"/>
+    <actuator name="motor3">
+      <hardwareInterface>EffortJointInterface</hardwareInterface>
+      <mechanicalReduction>1</mechanicalReduction>
+    </actuator>
+  </transmission>
+  <transmission name="tran4">
+    <type>transmission_interface/SimpleTransmission</type>
+    <joint name="${prefix}wrist_platform_joint"/>
+    <actuator name="motor4">
+      <hardwareInterface>EffortJointInterface</hardwareInterface>
+      <mechanicalReduction>1</mechanicalReduction>
+    </actuator>
+  </transmission>
+  <transmission name="tran5">
+    <type>transmission_interface/SimpleTransmission</type>
+    <joint name="${prefix}wrist_pitch_joint"/>
+    <actuator name="motor5">
+      <hardwareInterface>EffortJointInterface</hardwareInterface>
+      <mechanicalReduction>1</mechanicalReduction>
+    </actuator>
+  </transmission>
+  <transmission name="tran6">
+    <type>transmission_interface/SimpleTransmission</type>
+    <joint name="${prefix}wrist_yaw_joint"/>
+    <actuator name="motor6">
+      <hardwareInterface>EffortJointInterface</hardwareInterface>
+      <mechanicalReduction>1</mechanicalReduction>
+    </actuator>
+  </transmission>
+  <transmission name="tran7">
+    <type>transmission_interface/SimpleTransmission</type>
+    <joint name="${prefix}wrist_roll_joint"/>
+    <actuator name="motor7">
       <hardwareInterface>EffortJointInterface</hardwareInterface>
       <mechanicalReduction>1</mechanicalReduction>

Commit message: Added base and ee frames to the urdf to comply with ISI manual

File: dvrk_model/model/mtm.urdf.xacro (robot description, xacro)
@@ -298,74 +298,88 @@
       </inertial>
     </link>
-  <transmission name="tran1">
-    <type>transmission_interface/SimpleTransmission</type>
-    <joint name="${prefix}outer_yaw_joint"/>
-    <actuator name="motor1">
-      <hardwareInterface>EffortJointInterface</hardwareInterface>
-      <mechanicalReduction>1</mechanicalReduction>
-    </actuator>
-  </transmission>
-  <transmission name="tran2">
-    <type>transmission_interface/SimpleTransmission</type>
-    <joint name="${prefix}shoulder_pitch_joint"/>
-    <actuator name="motor2">
-      <hardwareInterface>EffortJointInterface</hardwareInterface>
-      <mechanicalReduction>1</mechanicalReduction>
-    </actuator>
-  </transmission>
-  <transmission name="tran3">
-    <type>transmission_interface/SimpleTransmission</type>
-    <joint name="${prefix}elbow_pitch_joint"/>
-    <actuator name="motor3">
-      <hardwareInterface>EffortJointInterface</hardwareInterface>
-      <mechanicalReduction>1</mechanicalReduction>
-    </actuator>
-  </transmission>
-  <transmission name="tran4">
-    <type>transmission_interface/SimpleTransmission</type>
-    <joint name="${prefix}wrist_platform_joint"/>
-    <actuator name="motor4">
-      <hardwareInterface>EffortJointInterface</hardwareInterface>
-      <mechanicalReduction>1</mechanicalReduction>
-    </actuator>
-  </transmission>
-  <transmission name="tran5">
-    <type>transmission_interface/SimpleTransmission</type>
-    <joint name="${prefix}wrist_pitch_joint"/>
-    <actuator name="motor5">
-      <hardwareInterface>EffortJointInterface</hardwareInterface>
-      <mechanicalReduction>1</mechanicalReduction>
-    </actuator>
-  </transmission>
-  <transmission name="tran6">
-    <type>transmission_interface/SimpleTransmission</type>
-    <joint name="${prefix}wrist_yaw_joint"/>
-    <actuator name="motor6">
-      <hardwareInterface>EffortJointInterface</hardwareInterface>
-      <mechanicalReduction>1</mechanicalReduction>
-    </actuator>
-  </transmission>
-  <transmission name="tran7">
-    <type>transmission_interface/SimpleTransmission</type>
-    <joint name="${prefix}wrist_roll_joint"/>
-    <actuator name="motor7">
-      <hardwareInterface>EffortJointInterface</hardwareInterface>
-      <mechanicalReduction>1</mechanicalReduction>
-    </actuator>
-  </transmission>
-  <gazebo>
-    <plugin name="gazebo_ros_control" filename="libgazebo_ros_control.so">
-      <robotNamespace>/mtm</robotNamespace>
-    </plugin>
-  </gazebo>
-  <gazebo>
-    <plugin name="force_torque_sensor" filename="libgazebo_ros_f3d.so" >
-      <bodyName>${prefix}bottom_parallel_link</bodyName>
-      <frameName>${prefix}bottom_parallel_link</frameName>
-      <topicName>/force_torque_feedback</topicName>
-      <alwaysOn>true</alwaysOn>
-      <updateRate>100.0</updateRate>
-    </plugin>
-  </gazebo>
+    <!-- add base link to match DVRK manual -->
+    <joint name="${prefix}base" type="fixed">
+      <parent link="${prefix}top_panel"/>
+      <child link="${prefix}base"/>
+      <origin rpy="0 0 0" xyz="0 0 -0.190"/>
+    </joint>
+    <link name="${prefix}base"/>
+    <!-- add ee link to match DVRK manual -->
+    <joint name="${prefix}end_effector" type="fixed">
+      <parent link="${prefix}wrist_roll_link"/>
+      <child link="${prefix}ee_link"/>
+      <origin rpy="0 ${PI} 0" xyz="0 0 0.039"/>
+    </joint>
+    <link name="${prefix}ee_link"/>
+    <transmission name="tran1">
+      <type>transmission_interface/SimpleTransmission</type>
+      <joint name="${prefix}outer_yaw_joint"/>
+      <actuator name="motor1">
+        <hardwareInterface>EffortJointInterface</hardwareInterface>
+        <mechanicalReduction>1</mechanicalReduction>
+      </actuator>
+    </transmission>
+    <transmission name="tran2">
+      <type>transmission_interface/SimpleTransmission</type>
+      <joint name="${prefix}shoulder_pitch_joint"/>
+      <actuator name="motor2">
+        <hardwareInterface>EffortJointInterface</hardwareInterface>
+        <mechanicalReduction>1</mechanicalReduction>
+      </actuator>
+    </transmission>
+    <transmission name="tran3">
+      <type>transmission_interface/SimpleTransmission</type>
+      <joint name="${prefix}elbow_pitch_joint"/>
+      <actuator name="motor3">
+        <hardwareInterface>EffortJointInterface</hardwareInterface>
+        <mechanicalReduction>1</mechanicalReduction>
+      </actuator>
+    </transmission>
+    <transmission name="tran4">
+      <type>transmission_interface/SimpleTransmission</type>
+      <joint name="${prefix}wrist_platform_joint"/>
+      <actuator name="motor4">
+        <hardwareInterface>EffortJointInterface</hardwareInterface>
+        <mechanicalReduction>1</mechanicalReduction>
+      </actuator>
+    </transmission>
+    <transmission name="tran5">
+      <type>transmission_interface/SimpleTransmission</type>
+      <joint name="${prefix}wrist_pitch_joint"/>
+      <actuator name="motor5">
+        <hardwareInterface>EffortJointInterface</hardwareInterface>
+        <mechanicalReduction>1</mechanicalReduction>
+      </actuator>
+    </transmission>
+    <transmission name="tran6">
+      <type>transmission_interface/SimpleTransmission</type>
+      <joint name="${prefix}wrist_yaw_joint"/>
+      <actuator name="motor6">
+        <hardwareInterface>EffortJointInterface</hardwareInterface>
+        <mechanicalReduction>1</mechanicalReduction>
+      </actuator>
+    </transmission>
+    <transmission name="tran7">
+      <type>transmission_interface/SimpleTransmission</type>
+      <joint name="${prefix}wrist_roll_joint"/>
+      <actuator name="motor7">
+        <hardwareInterface>EffortJointInterface</hardwareInterface>
+        <mechanicalReduction>1</mechanicalReduction>
+      </actuator>
+    </transmission>
+    <gazebo>
+      <plugin name="gazebo_ros_control" filename="libgazebo_ros_control.so">
+        <robotNamespace>/mtm</robotNamespace>
+      </plugin>
+    </gazebo>
+    <gazebo>
+      <plugin name="force_torque_sensor" filename="libgazebo_ros_f3d.so" >
+        <bodyName>${prefix}bottom_parallel_link</bodyName>
+        <frameName>${prefix}bottom_parallel_link</frameName>
+        <topicName>/force_torque_feedback</topicName>
+        <alwaysOn>true</alwaysOn>
+        <updateRate>100.0</updateRate>
+      </plugin>
+    </gazebo>
   </xacro:macro>
 </robot>
